File: pcb/TypeO-conn-1/TypeO-conn-1.kicad_sch (KiCad schematic)
At the start: 9 parts, among them J1 USB_C_Receptacle_USB2.0, J2 Conn_01x05_Male, SW1 SW_DIP_x01

Commit message: Reorganize
Parts:
- removed JP2, JP3: (no value), symbol Jumper:SolderJumper_2_Open
- added JP2: CC2, Jumper:SolderJumper-2_P1.3mm_Bridged_RoundedPad1.0x1.5mm, symbol Jumper:SolderJumper_2_Bridged
- added JP3: CC1, Jumper:SolderJumper-2_P1.3mm_Bridged_RoundedPad1.0x1.5mm, symbol Jumper:SolderJumper_2_Bridged
- J2: value Conn_01x05_Male -> (none); footprint Connector_PinHeader_2.54mm:PinHeader_1x05_P2.54mm_Vertical -> (none)
Connections:
- net at J1.A5 (CC1): now also JP3.1 (A)
- net at J1.B5 (CC2): now also JP2.1 (A)
- net at R1.2: now also JP2.2 (B)
- net at R2.2: now also JP3.2 (B)
Other:
- note added: "D+"
- note added: "D-"
- note added: "GND"
- note added: "ID"
- note added: "VBUS"
Changed lines of the file:
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@@
     (stroke (width 0) (type default) (color 0 0 0 0))
+  )
+  (text "D+" (at 153.67 92.71 0)
+    (effects (font (size 1.27 1.27)) (justify left bottom))
+  )
+  (text "VBUS" (at 153.67 97.79 0)
+    (effects (font (size 1.27 1.27)) (justify left bottom))
+  )
+  (text "D-" (at 153.67 95.25 0)
+    (effects (font (size 1.27 1.27)) (justify left bottom))
+  )
+  (text "GND" (at 153.67 87.63 0)
+    (effects (font (size 1.27 1.27)) (justify left bottom))
+  )
+  (text "ID" (at 153.67 90.17 0)
+    (effects (font (size 1.27 1.27)) (justify left bottom))
   )
   (symbol (lib_id "Connector:USB_C_Receptacle_USB2.0") (at 38.1 88.9 0) (unit 1)
@@
   )
   (symbol (lib_id "Connector:Conn_01x05_Male") (at 152.4 92.71 180) (unit 1)
-    (in_bom yes) (on_board yes) (fields_autoplaced)
-    (property "Reference" "J2" (id 0) (at 153.67 91.4399 0)
+    (in_bom yes) (on_board yes)
+    (property "Reference" "J2" (id 0) (at 135.89 86.36 0)
       (effects (font (size 1.27 1.27)) (justify right))
     )
-    (property "Value" "Conn_01x05_Male" (id 1) (at 153.67 93.9799 0)
+    (property "Value" "" (id 1) (at 135.89 83.82 0)
       (effects (font (size 1.27 1.27)) (justify right))
     )
-    (property "Footprint" "Connector_PinHeader_2.54mm:PinHeader_1x05_P2.54mm_Vertical" (id 2) (at 152.4 92.71 0)
+    (property "Footprint" "" (id 2) (at 152.4 92.71 0)
       (effects (font (size 1.27 1.27)) hide)
     )
@@
     (pin "2")
   )
-  (symbol (lib_id "Jumper:SolderJumper_2_Open") (at 57.15 81.28 0) (unit 1)
+  (symbol (lib_id "Jumper:SolderJumper_2_Bridged") (at 60.96 78.74 0) (unit 1)
     (in_bom yes) (on_board yes)
-    (property "Reference" "JP2" (id 0) (at 57.15 83.82 0)
+    (property "Reference" "JP3" (id 0) (at 60.96 76.2 0))
+    (property "Value" "CC1" (id 1) (at 64.77 77.47 0))
+    (property "Footprint" "Jumper:SolderJumper-2_P1.3mm_Bridged_RoundedPad1.0x1.5mm" (id 2) (at 60.96 78.74 0)
       (effects (font (size 1.27 1.27)) hide)
     )
-    (property "Value" "" (id 1) (at 57.15 83.82 0))
-    (property "Footprint" "" (id 2) (at 57.15 81.28 0)
-      (effects (font (size 1.27 1.27)) hide)
-    )
-    (property "Datasheet" "~" (id 3) (at 57.15 81.28 0)
+    (property "Datasheet" "~" (id 3) (at 60.96 78.74 0)
       (effects (font (size 1.27 1.27)) hide)
     )
@@
     (pin "2")
   )
-  (symbol (lib_id "Jumper:SolderJumper_2_Open") (at 60.96 78.74 0) (unit 1)
+  (symbol (lib_id "Jumper:SolderJumper_2_Bridged") (at 57.15 81.28 0) (unit 1)
     (in_bom yes) (on_board yes)
-    (property "Reference" "JP3" (id 0) (at 60.96 72.39 0))
-    (property "Value" "" (id 1) (at 60.96 76.2 0))
-    (property "Footprint" "" (id 2) (at 60.96 78.74 0)
+    (property "Reference" "JP2" (id 0) (at 57.15 83.82 0))
+    (property "Value" "CC2" (id 1) (at 53.34 80.01 0))
+    (property "Footprint" "Jumper:SolderJumper-2_P1.3mm_Bridged_RoundedPad1.0x1.5mm" (id 2) (at 57.15 81.28 0)
       (effects (font (size 1.27 1.27)) hide)
     )
-    (property "Datasheet" "~" (id 3) (at 60.96 78.74 0)
+    (property "Datasheet" "~" (id 3) (at 57.15 81.28 0)
       (effects (font (size 1.27 1.27)) hide)
     )
@@
     )
     (path "/14052b08-1222-4446-b6b4-b88f5dfa20a6"
-      (reference "J2") (unit 1) (value "Conn_01x05_Male") (footprint "Connector_PinHeader_2.54mm:PinHeader_1x05_P2.54mm_Vertical")
+      (reference "J2") (unit 1) (value "Pogo pin header") (footprint "Connector_PinHeader_2.54mm:PinHeader_1x05_P2.54mm_Vertical")
     )
     (path "/aa594b1f-fd74-46a0-a124-e1d2aed26358"
       (reference "JP1") (unit 1) (value "SolderJumper_2_Open") (footprint "Jumper:SolderJumper-2_P1.3mm_Open_TrianglePad1.0x1.5mm")
     )
-    (path "/407fae1f-316c-420a-89e6-21f138123cbe"
-      (reference "JP2") (unit 1) (value "CC2") (footprint "Jumper:SolderJumper-2_P1.3mm_Open_RoundedPad1.0x1.5mm")
+    (path "/9d633ee8-8475-4b98-9e52-fa792e13dae0"
+      (reference "JP2") (unit 1) (value "CC2") (footprint "Jumper:SolderJumper-2_P1.3mm_Bridged_RoundedPad1.0x1.5mm")
     )
-    (path "/a66a3b2f-f268-4e38-987e-b27ec003ce16"
-      (reference "JP3") (unit 1) (value "CC1") (footprint "Jumper:SolderJumper-2_P1.3mm_Open_RoundedPad1.0x1.5mm")
+    (path "/69903f53-f077-4ff8-a212-14c4305face7"
+      (reference "JP3") (unit 1) (value "CC1") (footprint "Jumper:SolderJumper-2_P1.3mm_Bridged_RoundedPad1.0x1.5mm")
     )
     (path "/7342cc82-e0e9-41f9-8b46-68197771b07f"
