File: typeO-conn/typeO-conn-rounded.kicad_pcb (KiCad board)
At the start: 2 copper layers, 16.5 x 28.8 mm, 6 parts, among them J1 USB_C_Receptacle_USB2.0, J2 829-22-005-20-001101

Commit message: Add rounded, updated date
Routing:
- net Net-(J1-PadB5): track 24.3 -> 23.4 mm
- net Net-(J1-PadA5): track 16.8 -> 16.3 mm

Commit message: Tweaks
Routing:
- net /GND: track 4.91 -> 5.54 mm
