File: typeO-conn/typeO-conn.kicad_pcb (KiCad board)
At the start: 2 copper layers, 16.5 x 28.8 mm, 6 parts, among them J1 USB_C_Receptacle_USB2.0, J2 829-22-005-20-001101

Commit message: Tweaks
Routing:
- net /GND: track 4.91 -> 5.54 mm
Changed lines of the file:
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@@
     (effects (font (size 0.5 0.5) (thickness 0.1)) (justify mirror))
   )
-  (gr_text "{dblquote}Plug in a keyboard you found at the dump{dblquote}" (at 130.938021 88.10179 90) (layer "F.SilkS")
+  (gr_text "{dblquote}Plug in a keyboard you found at the dump{dblquote}" (at 130.938021 88.41179 90) (layer "F.SilkS")
     (effects (font (size 0.6 0.5) (thickness 0.1075) italic) (justify left))
   )
@@
   (segment (start 128.038021 71.75179) (end 125.888021 73.90179) (width 0.25) (layer "F.Cu") (net 8))
   (segment (start 125.888021 73.90179) (end 125.888021 77.09) (width 0.25) (layer "F.Cu") (net 8))
-  (segment (start 129.338021 73.75179) (end 129.338021 71.75179) (width 0.25) (layer "F.Cu") (net 9))
-  (via (at 129.338021 73.75179) (size 0.8) (drill 0.4) (layers "F.Cu" "B.Cu") (free) (net 9))
+  (segment (start 129.338021 74.38179) (end 129.338021 71.75179) (width 0.25) (layer "F.Cu") (net 9))
+  (via (at 129.338021 74.38179) (size 0.8) (drill 0.4) (layers "F.Cu" "B.Cu") (free) (net 9))
   (segment (start 121.128967 82.43682) (end 121.128967 83.21176) (width 0.25) (layer "B.Cu") (net 9))
   (segment (start 121.163997 82.40179) (end 121.128967 82.43682) (width 0.25) (layer "B.Cu") (net 9))
@@
       )
     )
+  )
+  (zone (net 0) (net_name "") (layer "B.Cu") (hatch edge 0.508)
+    (connect_pads (clearance 0))
+    (min_thickness 0.254)
+    (keepout (tracks allowed) (vias allowed) (pads allowed ) (copperpour not_allowed) (footprints allowed))
+    (fill (thermal_gap 0.508) (thermal_bridge_width 0.508))
+    (polygon
+      (pts
+        (xy 131.568021 73.74179)
+        (xy 124.038021 73.74179)
+        (xy 124.038021 70.22179)
+        (xy 131.568021 70.22179)
+      )
+    )
